Commit message: Sync workspace changes (excludes RViz URDF and fake launch)

File: rebotarm_ros2/third_party/reBotArm_control_py/urdf/00-arm-rs_asm-v3/urdf/00-arm-rs_asm-v3.urdf (robot description, URDF)
Before this commit: robot 00-arm-rs_asm-v3, 10 links, 9 joints
Links:
- link base_link: geometry collision mesh filename=package://rebotarm_bringup/description/meshes_rs/base_link.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; visual mesh filename=package://rebotarm_bringup/description/meshes_rs/base_link.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
- link gripper_end: geometry collision mesh filename=package://rebotarm_bringup/description/meshes_rs/gripper_en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; visual mesh filename=package://rebotarm_bringup/description/meshes_rs/cnc7.STL
- link gripper_left: geometry collision mesh filename=package://rebotarm_bringup/description/meshes_rs/gripper_le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; visual mesh filename=package://rebotarm_bringup/description/meshes_rs/cnc_left.S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
- link gripper_right: geometry collision mesh filename=package://rebotarm_bringup/description/meshes_rs/gripper_ri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; visual mesh filename=package://rebotarm_bringup/description/meshes_rs/cnc_right.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
- link link1: geometry collision mesh filename=package://rebotarm_bringup/description/meshes_rs/link1.STL; visual mesh filename=package://rebotarm_bringup/description/meshes_rs/link1.STL
- link link2: mass 1.552 -> 1.972; geometry collision mesh filename=package://rebotarm_bringup/description/meshes_rs/link2.STL; visual mesh filename=package://rebotarm_bringup/description/meshes_rs/cnc2.STL
- link link3: mass 1.252 -> 1.062; geometry collision mesh filename=package://rebotarm_bringup/description/meshes_rs/link3.STL; visual mesh filename=package://rebotarm_bringup/description/meshes_rs/cnc3.STL
- link link4: mass 0.46 -> 0.66; geometry collision mesh filename=package://rebotarm_bringup/description/meshes_rs/link4.STL; visual mesh filename=package://rebotarm_bringup/description/meshes_rs/cnc4.STL
- link link5: mass 0.20120457182895 -> 0.150120457182895; geometry collision mesh filename=package://rebotarm_bringup/description/meshes_rs/link5.STL; visual mesh filename=package://rebotarm_bringup/description/meshes_rs/cnc5.STL
- link link6: mass 0.1 -> 0.03; geometry collision mesh filename=package://rebotarm_bringup/description/meshes_rs/link6.STL; visual mesh filename=package://rebotarm_bringup/description/meshes_rs/link6.STL
Joints:
- removed joint joint_left
- removed joint joint_right
- added joint gripper_joint1: type prismatic, parent gripper_end, child gripper_left, origin xyz=-0.041939 -7.3385E-05 0 rpy=1.5708 -1.5708 0, axis 0 0 1, limit lower=0 upper=0.05 effort=500 velocity=10
- added joint gripper_joint2: type prismatic, parent gripper_end, child gripper_right, origin xyz=-0.041939 7.3385E-05 0 rpy=-1.5708 -1.5708 0, axis 0 0 1, limit lower=0 upper=0.0715 effort=500 velocity=10
